File: KiCad/RGBChain/RGBChain.kicad_pcb (KiCad board)
At the start: 2 copper layers, 95 x 90 mm, 72 parts, among them J1 AudioJack2_Ground, J2 SWD, J3 USB_B_Micro, J4 Barrel_Jack, P1 USB_C_Plug_USB2.0, Q1 IRF7404, Q2 SQJB80EP, Q3 IRLML2502, SW1 Rotary_Encoder_Switch, SW2 SW_SPDT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

Commit message: PCB done
Parts:
- added D7: RED LED, LED_THT:LED_D3.0mm, F.Cu at (94.0, 85.4)
- added D8: RED LED, LED_THT:LED_D3.0mm, F.Cu at (94.0, 93.0)
- D6: value WS2812B -> WS2812D; footprint LED_THT:LED_D5.0mm-4_RGB_Staggered_Pins -> LED_THT:LED_D5.0mm-4_RGB
- J1: footprint Connector_Audio:Jack_3.5mm_CUI_SJ-3523-SMT_Horizontal -> JPConnectors:Jack_3.5mm_Lumberg_1503_03
- JP1: moved to B.Cu
- SW2: footprint Button_Switch_THT:SW_E-Switch_EG1224_SPDT_Angled -> JPSwitches:NINIGI_5F_M6
- moved D2 13.1 mm to (96.2, 86.8)
- moved R1 7.73 mm to (92.0, 86.8), turned to 90 degrees
- moved D3 6.97 mm to (96.2, 94.2)
- moved D1 6.48 mm to (86.8, 93.0), turned to 270 degrees
- moved J1 6.40 mm to (109.3, 40.1)
- moved JP1 4.83 mm to (81.2, 71.8)
- moved R7 3.47 mm to (91.8, 94.2), turned to 90 degrees
- moved SW2 2.56 mm to (22.2, 62.2)
- moved C4 2.33 mm to (55.4, 88.4)
- moved C1 0.92 mm to (81.1, 75.0)
- moved L2 0.90 mm to (73.6, 42.4)
- moved Q2 0.90 mm to (64.0, 85.0)
- moved R2 0.80 mm to (54.1, 84.8)
- moved BT3 0.49 mm to (57.4, 64.9)
- moved C2 0.41 mm to (89.2, 85.0)
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Connections:
- D6 pad 1: +5V -> Net-(D6-Pad1)
- D6 pad 2: Net-(D6-Pad2) -> +5V
Routing:
- net +BATT: track 111.8 -> 180.2 mm, vias 3 -> 2
- net GNDPWR: track 75.6 -> 122.0 mm, vias 14 -> 20
- net VBUS: track 32.5 -> 43.8 mm, vias 1 -> 2
- net +5V: track 77.2 -> 83.6 mm, vias 0 -> 1
- net Net-(R7-Pad1): track 6.96 -> 12.7 mm
- net Net-(C2-Pad1): track 18.2 -> 23.2 mm
- net Net-(D6-Pad4): track 14.5 -> 18.9 mm, vias 0 -> 1
- net POWER: track 85.6 -> 89.4 mm
- net -BATT: track 69.1 -> 72.4 mm, vias 1 -> 2
- net Net-(D3-Pad1): track 1.53 -> 4.62 mm
- net GND: track 25.7 -> 28.7 mm
- net Net-(D2-Pad1): track 1.53 -> 4.58 mm
- net +3V3: track 75.1 -> 74.1 mm
- net Net-(Q2-Pad4): track 2.09 -> 2.99 mm
- net +3.3VA: track 9.09 -> 8.19 mm
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Other:
- board text added: "+3v3"
- board text added: "Charging"
- board text added: "GND"
- board text added: "NRST"
- board text added: "Power"
- board text added: "RGB Chain v1 JP, 2020.10.24"
- board text added: "SWCLK"
- board text added: "SWD"
- board text added: "SWDIO"

Commit message: PCB more work
Parts:
- removed JP1: 0, Jumper:SolderJumper-2_P1.3mm_Bridged_Pad1.0x1.5mm
- BT1, BT2, BT3: footprint Battery:BatteryHolder_Keystone_1042_1x18650 -> JPConnectors:BatteryHolder_Keystone_1042_1x18650
- R10, R4: footprint Resistor_SMD:R_0805_2012Metric -> Resistor_SMD:R_0603_1608Metric
- U5: value STM32L051K8Tx -> STM32L051K8T6
- moved C1 26.3 mm to (57.9, 62.7), turned to 270 degrees
- moved U1 21.8 mm to (61.3, 62.8), turned to 0 degrees
- moved C3 16.5 mm to (64.7, 62.7), turned to 270 degrees
Connections:
- C1 pad 2: GNDPWR -> GND
- C12 pad 2: GNDPWR -> GND
- C14 pad 2: GNDPWR -> GND
- C15 pad 2: GNDPWR -> GND
- C19 pad 2: GNDPWR -> GND
- C2 pad 2: GNDPWR -> GND
- C5 pad 2: GNDPWR -> GND
- C6 pad 2: GNDPWR -> GND
- C7 pad 2: GNDPWR -> GND
- C8 pad 2: GNDPWR -> GND
- D6 pad 3: GNDPWR -> GND
- J1 pad G: GNDPWR -> GND
- J3 pad 5: GNDPWR -> GND
- J4 pad 2: GNDPWR -> GND
- P1 pad A1: GNDPWR -> GND
- P1 pad A12: GNDPWR -> GND
- P1 pad B1: GNDPWR -> GND
- P1 pad B12: GNDPWR -> GND
- Q2 pad 1: GNDPWR -> GND
- R1 pad 1: GNDPWR -> GND
- R5 pad 1: GNDPWR -> GND
- R9 pad 2: GNDPWR -> GND
- U1 pad 4: Net-(U1-Pad4) -> GND
- U3 pad 6: GNDPWR -> GND
- U4 pad 2: GNDPWR -> GND
Routing:
- net GND: track 28.7 -> 152.5 mm, vias 13 -> 35
- net GNDPWR: track 122.0 -> 0.00 mm, vias 20 -> 0
- net POWER: track 89.4 -> 66.8 mm
- net +3V3: track 74.1 -> 69.6 mm
- net VBUS: track 43.8 -> 44.1 mm, vias 2 -> 5
- removed copper zone on B.Cu, net GNDPWR
Other:
- board text added: "."
- board text added: "STM32L051K8T6"

Commit message: Last pcb changes
Parts:
- J2: footprint Connector_PinHeader_2.54mm:PinHeader_1x06_P2.54mm_Vertical -> Connector_PinHeader_2.54mm:PinHeader_1x05_P2.54mm_Vertical
- J4: value Barrel_Jack -> Power
- P1: footprint Connector_USB:USB_C_Receptacle_Amphenol_12401610E4-2A -> JPConnectors:USB_C_Receptacle_Adam_Tech; moved to B.Cu
- moved P1 9.55 mm to (103.4, 79.4), turned to 270 degrees
- moved SW1 9.50 mm to (98.0, 70.5)
- moved C8 5.80 mm to (73.2, 81.6), turned to 270 degrees
- moved D8 2.60 mm to (94.0, 95.6), turned to 90 degrees
- moved J2 2.16 mm to (95.4, 50.0), turned to 270 degrees
- moved Q1 0.60 mm to (78.3, 85.2)
- moved J3 0.30 mm to (107.0, 92.4)
- moved BT2 0.22 mm to (80.0, 65.0)
- turned D3 to 90 degrees
- turned R7 to 270 degrees
Connections:
- D3 pad 2: VBUS -> Net-(C2-Pad1)
- D8 pad 2: VBUS -> Net-(C2-Pad1)
Routing:
- net VBUS: track 44.1 -> 61.8 mm, vias 5 -> 10
- net Net-(P1-PadS1): track 0.00 -> 9.43 mm
- net NRST: track 27.0 -> 35.8 mm
- net Net-(C2-Pad1): track 23.2 -> 30.3 mm
- net Net-(R17-Pad1): track 23.7 -> 18.2 mm
- net SWDIO: track 15.5 -> 20.9 mm
- net Net-(R14-Pad1): track 40.3 -> 36.2 mm
- net Net-(R13-Pad1): track 41.8 -> 37.9 mm
- net SWCLK: track 11.7 -> 13.9 mm
- net GND: track 152.5 -> 150.3 mm, vias 35 -> 32
- net Net-(R7-Pad1): track 12.7 -> 10.8 mm
- net +BATT: track 180.2 -> 178.7 mm
- net POWER: track 66.8 -> 65.6 mm, vias 4 -> 6
- added copper zone on F.Cu, net GND
Other:
- outline, holes or cut-outs redrawn
- net class Default: clearance 0.15 -> 0.12
- rule trace_clearance: 0.15 -> 0.12
- board text added: "Charging limit by R3 (2512) Limit | R3 | Pmax / R3 500mA | 220m | 66mW 1A | 110m | 131mW 2A | 55m | 240mW"
- board text added: "RGB Chain v1 JP, 2020.11.4"
- board text removed: "RGB Chain v1 JP, 2020.10.24"

Commit message: More effects. Refactoring
Changed lines of the file:
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@@
   )
   (setup
-    (last_trace_width 0.6)
+    (last_trace_width 0.25)
     (user_trace_width 0.28)
     (user_trace_width 0.4)
@@
     (tags resistor)
     (attr smd)
-    (fp_text reference R12 (at 0 -3.6) (layer F.SilkS)
+    (fp_text reference R12 (at 0 1.6) (layer F.SilkS)
       (effects (font (size 1 1) (thickness 0.15)))
     )
@@
     (tags diode)
     (attr smd)
-    (fp_text reference D5 (at 0 -3.6) (layer F.SilkS)
-      (effects (font (size 1 1) (thickness 0.15)))
-    )
+    (fp_text reference D5 (at 0 1.8) (layer F.SilkS)
+      (effects (font (size 1 1) (thickness 0.15)))
+    )
